File: Corinthians-Flight-Control-System-PCB/_autosave-Corinthians-Flight-Control-System.kicad_pcb (KiCad board)
At the start: 4 copper layers, 48.9 x 72.5 mm, 83 parts, among them J0 RaspberryPi, J1 50ohm Coaxial Ant, J10 M8, J11 M9, J12 M10, J2 GPS/Compass, J3 M1, J4 M2, J5 M3, J6 M4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

Commit message: Post DRC Check
Parts:
- moved C18 1.72 mm to (118.7, 164.7)
- moved D6 0.72 mm to (110.6, 125.8)
- moved F1 0.42 mm to (114.7, 125.8)
- moved FB1 0.14 mm to (118.7, 125.8)
Routing:
- net +5V: track 11.2 -> 9.07 mm
- net Net-(C18-Pad2): track 3.26 -> 4.55 mm
- net GND: track 112.7 -> 113.8 mm
- net Net-(C26-Pad1): track 9.33 -> 9.93 mm
