File: Corinthians-Flight-Control-System-PCB/Corinthians-Flight-Control-System.kicad_pcb (KiCad board)
At the start: 4 copper layers, 48.9 x 72.5 mm, 83 parts, among them J0 RaspberryPi, J1 50ohm Coaxial Ant, J10 M8, J11 M9, J12 M10, J2 GPS/Compass, J3 M1, J4 M2, J5 M3, J6 M4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

Commit message: clean
Routing:
- net Net-(C1-Pad2): track 13.0 -> 12.3 mm
